Commit message: Add files via upload

File: Kinematic_Scenes/scenes/NEXXUS_ROV.urdf (robot description, URDF)
Before this commit: robot NEXXUS_ROV, 19 links, 18 joints
Links:
- removed link bottom_left_finger
- removed link bottom_right_finger
- removed link inner_rotate_left
- removed link inner_rotate_wrist_right
- removed link left_base
- removed link long_arm_left
- removed link long_arm_right
- removed link middle_left_finger
- removed link middle_right_finger
- removed link outer_rotate_left
- removed link outer_wrist_right
- removed link right_base
- removed link short_arm_left
- removed link short_arm_right
- removed link top_left_finger
- removed link top_right_finger
- removed link wrist_left
- removed link wrist_right
- added link left1; collision mesh filename=/home/burobotics/catkin_ws/src/NEXXUS_ROV/meshes/left1.STL; visual mesh filename=/home/burobotics/catkin_ws/src/NEXXUS_ROV/meshes/left1.STL
- added link left2; collision mesh filename=/home/burobotics/catkin_ws/src/NEXXUS_ROV/meshes/left2.STL; visual mesh filename=/home/burobotics/catkin_ws/src/NEXXUS_ROV/meshes/left2.STL
- added link left3; collision mesh filename=/home/burobotics/catkin_ws/src/NEXXUS_ROV/meshes/left3.STL; visual mesh filename=/home/burobotics/catkin_ws/src/NEXXUS_ROV/meshes/left3.STL
- added link left4; collision mesh filename=/home/burobotics/catkin_ws/src/NEXXUS_ROV/meshes/left4.STL; visual mesh filename=/home/burobotics/catkin_ws/src/NEXXUS_ROV/meshes/left4.STL
- added link left5; collision mesh filename=/home/burobotics/catkin_ws/src/NEXXUS_ROV/meshes/left5.STL; visual mesh filename=/home/burobotics/catkin_ws/src/NEXXUS_ROV/meshes/left5.STL
- added link left6; collision mesh filename=/home/burobotics/catkin_ws/src/NEXXUS_ROV/meshes/left6.STL; visual mesh filename=/home/burobotics/catkin_ws/src/NEXXUS_ROV/meshes/left6.STL
- added link left_F_1; collision mesh filename=/home/burobotics/catkin_ws/src/NEXXUS_ROV/meshes/left_F_1.S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; visual mesh filename=/home/burobotics/catkin_ws/src/NEXXUS_ROV/meshes/left_F_1.S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
- added link left_F_2; collision mesh filename=/home/burobotics/catkin_ws/src/NEXXUS_ROV/meshes/left_F_2.S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; visual mesh filename=/home/burobotics/catkin_ws/src/NEXXUS_ROV/meshes/left_F_2.S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
- added link right1; collision mesh filename=/home/burobotics/catkin_ws/src/NEXXUS_ROV/meshes/right1.STL; visual mesh filename=/home/burobotics/catkin_ws/src/NEXXUS_ROV/meshes/right1.STL
- added link right2; collision mesh filename=/home/burobotics/catkin_ws/src/NEXXUS_ROV/meshes/right2.STL; visual mesh filename=/home/burobotics/catkin_ws/src/NEXXUS_ROV/meshes/right2.STL
- added link right3; collision mesh filename=/home/burobotics/catkin_ws/src/NEXXUS_ROV/meshes/right3.STL; visual mesh filename=/home/burobotics/catkin_ws/src/NEXXUS_ROV/meshes/right3.STL
- added link right4; collision mesh filename=/home/burobotics/catkin_ws/src/NEXXUS_ROV/meshes/right4.STL; visual mesh filename=/home/burobotics/catkin_ws/src/NEXXUS_ROV/meshes/right4.STL
- added link right5; collision mesh filename=/home/burobotics/catkin_ws/src/NEXXUS_ROV/meshes/right5.STL; visual mesh filename=/home/burobotics/catkin_ws/src/NEXXUS_ROV/meshes/right5.STL
- added link right6; collision mesh filename=/home/burobotics/catkin_ws/src/NEXXUS_ROV/meshes/right6.STL; visual mesh filename=/home/burobotics/catkin_ws/src/NEXXUS_ROV/meshes/right6.STL
- added link right_F_1; collision mesh filename=/home/burobotics/catkin_ws/src/NEXXUS_ROV/meshes/right_F_1.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; visual mesh filename=/home/burobotics/catkin_ws/src/NEXXUS_ROV/meshes/right_F_1.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
- added link right_F_2; collision mesh filename=/home/burobotics/catkin_ws/src/NEXXUS_ROV/meshes/right_F_2.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; visual mesh filename=/home/burobotics/catkin_ws/src/NEXXUS_ROV/meshes/right_F_2.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
- link base_link: mass 7776.50474086467 -> 7776; geometry collision mesh filename=/home/burobotics/catkin_ws/src/NEXXUS_ROV/meshes/base_link.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; visual mesh filename=/home/burobotics/catkin_ws/src/NEXXUS_ROV/meshes/base_link.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
Joints:
- removed joint bottom_hand_left
- removed joint inner_wrist_right
- removed joint left_arm_rotate
- removed joint left_base_to_long_arm
- removed joint left_wrist_rotate
- removed joint long_arm_to_base_right
- removed joint long_to_short_left
- removed joint long_to_short_right
- removed joint middle_hand_left
- removed joint right_arm_rotate
- removed joint right_hand_bottom
- removed joint right_hand_middle
- removed joint right_hand_top
- removed joint right_wrist_rotate
- removed joint short_to_wrist_left
- removed joint short_to_wrist_right
- removed joint top_hand_left
- removed joint wrist_to_rotate_left
- added joint left1: type continuous, parent base_link, child left1, origin xyz=1.275 -0.4734 0.064987 rpy=-1.5708 -6.123E-17 -1.5708, axis 0 -1 0, limit lower=-1 upper=1 effort=0 velocity=0
- added joint left2: type continuous, parent left1, child left2, origin xyz=0 -0.18 0.1 rpy=0 -1.5708 0, axis 0 0 1, limit lower=-1 upper=1 effort=0 velocity=0
- added joint left3: type continuous, parent left2, child left3, origin xyz=0.75 0 0 rpy=0 0 0, axis 0 0 1, limit lower=-1 upper=1 effort=0 velocity=0
- added joint left4: type continuous, parent left3, child left4, origin xyz=0.55 0 0 rpy=0 0 0, axis 0 0 1, limit lower=-1 upper=1 effort=0 velocity=0
- added joint left5: type continuous, parent left4, child left5, origin xyz=0.15 0 0 rpy=1.5708 0 0, axis 0 0 -1, limit lower=-1 upper=1 effort=0 velocity=0
- added joint left6: type continuous, parent left5, child left6, origin xyz=0.25 0 0 rpy=0 0 0, axis 1 0 0, limit lower=-1 upper=1 effort=0 velocity=0
- added joint left_F_1: type continuous, parent left6, child left_F_1, origin xyz=0.2 0 0 rpy=1.5708 -2.7756E-15 -1.5708, axis 0 -1 0, limit lower=-1 upper=1 effort=0 velocity=0
- added joint left_F_2: type continuous, parent left6, child left_F_2, origin xyz=0.2 0 0 rpy=1.5708 2.7756E-15 1.5708, axis 0 -1 0, limit lower=-1 upper=1 effort=0 velocity=0
- added joint right1: type continuous, parent base_link, child right1, origin xyz=1.2551 0.49063 0.064987 rpy=-1.5708 -6.123E-17 -1.5708, axis 0 -1 0, limit lower=-1 upper=1 effort=0 velocity=0
- added joint right2: type continuous, parent right1, child right2, origin xyz=0 -0.18 0.1 rpy=0 -1.5708 0, axis 0 0 1, limit lower=-1 upper=1 effort=0 velocity=0
- added joint right3: type continuous, parent right2, child right3, origin xyz=0.75 0 0 rpy=0 0 0, axis 0 0 1, limit lower=-1 upper=1 effort=0 velocity=0
- added joint right4: type continuous, parent right3, child right4, origin xyz=0.55 0 0 rpy=0 0 0, axis 0 0 1, limit lower=-1 upper=1 effort=0 velocity=0
- added joint right5: type continuous, parent right4, child right5, origin xyz=0.15 0 0 rpy=1.5708 0 0, axis 0 0 -1, limit lower=-1 upper=1 effort=0 velocity=0
- added joint right6: type continuous, parent right5, child right6, origin xyz=0.25 0 0 rpy=0 0 0, axis 1 0 0, limit lower=-1 upper=1 effort=0 velocity=0
- added joint right_F_1: type continuous, parent right6, child right_F_1, origin xyz=0.2 0 0 rpy=1.5708 0 1.5708, axis 0 -1 0, limit lower=-1 upper=1 effort=0 velocity=0
- added joint right_F_2: type continuous, parent right6, child right_F_2, origin xyz=0.2 0 0 rpy=1.6501 -1.1177E-08 -1.5708, axis 0 -0.99685 0.079255, limit lower=-1 upper=1 effort=0 velocity=0
